File: sprig-hax/hardware/DebugShimPCB/pico-reset.kicad_sch (KiCad schematic)
At the start: 3 parts, among them J2 PINHD_1x3_Female, SW1 Push_Button

Commit message: updated data for parts
Parts:
- J2: LCSC (none) -> C2897385
- SW1: LCSC (none) -> C6748648
Changed lines of the file:
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@@
+      (effects (font (size 1.27 1.27)) hide)
+    )
+    (property "LCSC" "C6748648" (at 168.91 97.79 0)
       (effects (font (size 1.27 1.27)) hide)
     )
@@
       (effects (font (size 1.27 1.27)) hide)
     )
+    (property "LCSC" "C2897385" (at 93.98 77.47 0)
+      (effects (font (size 1.27 1.27)) hide)
+    )
